File: dev-board-1.0/mokki-dev-board/mokki-dev-board.sch (KiCad schematic (older format))
At the start: 43 parts

Commit message: Fixed LED - common anode, removed multiple labels, added values to some components
Parts:
- removed C? (x5): C, symbol Device:C
- added C? (x5): 100n, symbol Device:C_Small
- C? (x2): value C_Small -> 22p
- C?: value C -> 10u
- C?: value C_Small -> 100n
- C? (x2): value C_Small -> 100p
- Q?: value Q_NPN_CBE -> BC847B
- R? (x2): value R_Small -> 22R
- R?: value R_Small -> 10K
- R? (x3): value R_Small -> 50R
- R?: value R_Small -> 1k
- Y?: value Crystal_Small -> 12M0
- Y?: value Crystal_Small -> 32k768
Connections:
- net labels added: VDD, VSS
- net labels removed: VDD1, VDD2, VDD3, VDD4, VDDA, VSS1, VSS2, VSS3, VSS4, VSSA
- wire segments 249 -> 265
Other:
- note added: "Capacitors close to VDD/VSS pins"
- note added: "Common anode (60 mA)"
- moved on the sheet: BT?, C?, D?, LS?, Q?, R?, SW?, Y?

Commit message: missing wire
Connections:
- wire segments 265 -> 266
Changed lines of the file:
@@
 Wire Wire Line
 	1050 3300 1050 3350
+Wire Wire Line
+	10350 4850 10350 5450
 $EndSCHEMATC

Commit message: Footprints assigned
Parts:
- BT1: renamed from BT?; footprint (none) -> TestPoint:TestPoint_2Pads_Pitch2.54mm_Drill0.8mm
- C1, C2, C3, C4: renamed from C?; footprint (none) -> Capacitor_SMD:C_0603_1608Metric_Pad1.05x0.95mm_HandSolder
- C10, C11, C5, C6, C7, C8, C9: renamed from C?; footprint (none) -> Capacitor_SMD:C_0805_2012Metric_Pad1.15x1.40mm_HandSolder
- D1: renamed from D?; footprint (none) -> LED_SMD:LED_RGB_5050-6
- J1: renamed from J?; footprint (none) -> Connector_USB:USB_Micro-B_Molex_47346-0001
- J2: renamed from J?; footprint (none) -> Connector_PinSocket_2.54mm:PinSocket_1x04_P2.54mm_Horizontal
- J3: renamed from J?; footprint (none) -> Connector_PinSocket_2.54mm:PinSocket_1x04_P2.54mm_Vertical
- J4: renamed from J?; footprint (none) -> Connector_PinSocket_2.54mm:PinSocket_1x06_P2.54mm_Horizontal
- J5: renamed from J?; footprint (none) -> Connector_PinSocket_2.54mm:PinSocket_1x02_P2.54mm_Horizontal
- J6: renamed from J?; footprint (none) -> Connector_PinSocket_2.54mm:PinSocket_2x20_P2.54mm_Horizontal
- LS1: renamed from LS?; footprint (none) -> Connector_PinHeader_1.00mm:PinHeader_1x02_P1.00mm_Vertical
- Q1: renamed from Q?; footprint (none) -> Package_TO_SOT_SMD:SOT-23_Handsoldering
- R1, R2, R3, R4, R5, R6, R7, R8, R9: renamed from R?; footprint (none) -> Resistor_SMD:R_0805_2012Metric_Pad1.15x1.40mm_HandSolder
- SW1: renamed from SW?; value SW_SPST -> SW_PWR; footprint (none) -> Connector_PinHeader_2.54mm:PinHeader_1x03_P2.54mm_Horizontal
- SW10, SW3, SW4, SW5, SW7, SW8, SW9: renamed from SW?; footprint (none) -> Button_Switch_SMD:SW_SPST_TL3305B
- SW2: renamed from SW?; value SW_SPST -> BTN_RST; footprint (none) -> Button_Switch_SMD:SW_SPST_TL3305B
- SW6: renamed from SW?; footprint (none) -> Button_Switch_THT:SW_Tactile_SPST_Angled_PTS645Vx58-2LFS
- Y1: renamed from Y?; footprint (none) -> Crystal:Crystal_SMD_5032-2Pin_5.0x3.2mm_HandSoldering
- Y2: renamed from Y?; footprint (none) -> Crystal:Crystal_C38-LF_D3.0mm_L8.0mm_Horizontal
- gave numbers to parts that had none: 1
Connections:
- net labels removed: SPI3_CK, USART4_RX, USART4_TX

Commit message: Fixed user port issue
Parts:
- removed J6: User port (female), Connector_PinSocket_2.54mm:PinSocket_2x20_P2.54mm_Horizontal, symbol Connector_Generic:Conn_02x20_Row_Letter_First
- added J6: User port, Connector_PinSocket_2.54mm:PinSocket_2x20_P2.54mm_Horizontal, symbol Connector_Generic:Conn_02x20_Odd_Even
Changed lines of the file:
@@
 	8350 2750 8350 2800
-Wire Wire Line
-	8350 2800 8850 2800
 Wire Wire Line
 	8850 2800 8850 2750
@@
 Wire Wire Line
 	8350 2800 8350 2850
-Wire Wire Line
-	8850 2800 9350 2800
 Wire Wire Line
 	9350 2800 9350 2750
@@
 	6800 5500 7250 5500
 Wire Wire Line
-	6800 5000 7250 5000
-Wire Wire Line
 	6650 5050 6650 5100
-Wire Wire Line
-	6650 5100 7250 5100
 Wire Wire Line
 	7250 5200 6650 5200
@@
 Wire Notes Line
 	8050 5650 6500 5650
-$Comp
-L Connector_Generic:Conn_02x20_Row_Letter_First J6
-U 1 1 5BEAA45F
-P 9850 4650
-F 0 "J6" V 9946 5630 50  0000 L CNN
-F 1 "User port (female)" V 9855 5630 50  0000 L CNN
-F 2 "Connector_PinSocket_2.54mm:PinSocket_2x20_P2.54mm_Horizontal" H 9850 4650 50  0001 C CNN
-F 3 "~" H 9850 4650 50  0001 C CNN
-	1    9850 4650
-	0    -1   -1   0
-$EndComp
 Text Notes 10950 6250 2    50   ~ 0
 a - upper row / b - lower row\nA - analog input\nT - timer (PWM output)
@@
 Text Label 9650 5450 1    50   ~ 0
 GPIO_PC8_T
-Wire Wire Line
-	9150 5450 9150 4850
 Wire Wire Line
 	9250 5450 9250 4850
@@
 Wire Wire Line
 	9850 4850 9850 5700
-Wire Wire Line
-	9850 5700 9750 5700
 Connection ~ 9750 5700
-Wire Wire Line
-	8950 4850 8950 5700
-Wire Wire Line
-	9050 4850 9050 5700
 Connection ~ 9050 5700
 Wire Wire Line
@@
 Wire Wire Line
 	8950 3500 8700 3500
-Wire Wire Line
-	8700 3500 8700 3600
-Wire Wire Line
-	8950 3500 9050 3500
-Wire Wire Line
-	9050 3500 9050 4350
 Connection ~ 8950 3500
 Wire Wire Line
-	9050 3500 9750 3500
-Wire Wire Line
 	9750 3500 9750 4350
-Connection ~ 9050 3500
 Wire Wire Line
 	9750 3500 9850 3500
@@
 Wire Wire Line
 	10450 4850 10450 5700
-Wire Wire Line
-	10450 5700 9850 5700
 Connection ~ 9850 5700
 Text Label 10550 5450 1    50   ~ 0
@@
 Wire Wire Line
 	10350 4850 10350 5450
+$Comp
+L Connector_Generic:Conn_02x20_Odd_Even J6
+U 1 1 5B61C644
+P 9950 4650
+F 0 "J6" V 10050 3450 50  0000 L CNN
+F 1 "User port" V 9950 3200 50  0000 L CNN
+F 2 "Connector_PinSocket_2.54mm:PinSocket_2x20_P2.54mm_Horizontal" H 9950 4650 50  0001 C CNN
+F 3 "~" H 9950 4650 50  0001 C CNN
+	1    9950 4650
+	0    1    -1   0
+$EndComp
+Wire Wire Line
+	9150 4850 9150 5450
+Wire Wire Line
+	8950 4850 8950 5700
+Wire Wire Line
+	8350 2800 8850 2800
+Wire Wire Line
+	8850 2800 9350 2800
+Wire Wire Line
+	9750 5700 9850 5700
+Wire Wire Line
+	9850 5700 10450 5700
+Wire Wire Line
+	8700 3500 8700 3600
+Wire Wire Line
+	8950 3500 9050 3500
+Wire Wire Line
+	9050 4350 9050 3500
+Connection ~ 9050 3500
+Wire Wire Line
+	9050 3500 9750 3500
+Wire Wire Line
+	9050 4850 9050 5700
+Wire Wire Line
+	6800 5000 7250 5000
+Wire Wire Line
+	6650 5100 7250 5100
 $EndSCHEMATC

Commit message: Modified some footprints, used 0603 capacitors
Parts:
- C10, C11, C5, C6, C7, C8: footprint Capacitor_SMD:C_0805_2012Metric_Pad1.15x1.40mm_HandSolder -> Capacitor_SMD:C_0603_1608Metric_Pad1.05x0.95mm_HandSolder
- LS1: footprint Connector_PinHeader_1.00mm:PinHeader_1x02_P1.00mm_Vertical -> TestPoint:tp-smd-2pad
- R1, R2: footprint Resistor_SMD:R_0805_2012Metric_Pad1.15x1.40mm_HandSolder -> Resistor_SMD:R_0603_1608Metric_Pad1.05x0.95mm_HandSolder
Changed lines of the file:
@@
 F 0 "R1" V 1004 2950 50  0000 C CNN
 F 1 "R_Small" V 1095 2950 50  0000 C CNN
-F 2 "Resistor_SMD:R_0805_2012Metric_Pad1.15x1.40mm_HandSolder" H 1200 2950 50  0001 C CNN
+F 2 "Resistor_SMD:R_0603_1608Metric_Pad1.05x0.95mm_HandSolder" H 1200 2950 50  0001 C CNN
 F 3 "~" H 1200 2950 50  0001 C CNN
 	1    1200 2950
@@
 F 0 "C11" H 7092 1296 50  0000 L CNN
 F 1 "100n" H 7092 1205 50  0000 L CNN
-F 2 "Capacitor_SMD:C_0805_2012Metric_Pad1.15x1.40mm_HandSolder" H 7000 1250 50  0001 C CNN
+F 2 "Capacitor_SMD:C_0603_1608Metric_Pad1.05x0.95mm_HandSolder" H 7000 1250 50  0001 C CNN
 F 3 "~" H 7000 1250 50  0001 C CNN
 	1    7000 1250
@@
 F 0 "R2" V 1004 4750 50  0000 C CNN
 F 1 "R_Small" V 1095 4750 50  0000 C CNN
-F 2 "Resistor_SMD:R_0805_2012Metric_Pad1.15x1.40mm_HandSolder" H 1200 4750 50  0001 C CNN
+F 2 "Resistor_SMD:R_0603_1608Metric_Pad1.05x0.95mm_HandSolder" H 1200 4750 50  0001 C CNN
 F 3 "~" H 1200 4750 50  0001 C CNN
 	1    1200 4750
@@
 F 0 "LS1" H 6070 4596 50  0000 L CNN
 F 1 "Speaker" H 6070 4505 50  0000 L CNN
-F 2 "Connector_PinHeader_1.00mm:PinHeader_1x02_P1.00mm_Vertical" H 5900 4400 50  0001 C CNN
+F 2 "TestPoint:tp-smd-2pad" H 5900 4400 50  0001 C CNN
 F 3 "~" H 5890 4550 50  0001 C CNN
 	1    5900 4600
@@
 F 0 "C5" H 4992 2496 50  0000 L CNN
 F 1 "100n" H 4992 2405 50  0000 L CNN
-F 2 "Capacitor_SMD:C_0805_2012Metric_Pad1.15x1.40mm_HandSolder" H 4900 2450 50  0001 C CNN
+F 2 "Capacitor_SMD:C_0603_1608Metric_Pad1.05x0.95mm_HandSolder" H 4900 2450 50  0001 C CNN
 F 3 "~" H 4900 2450 50  0001 C CNN
 	1    4900 2450
@@
 F 0 "C6" H 5292 2496 50  0000 L CNN
 F 1 "100n" H 5292 2405 50  0000 L CNN
-F 2 "Capacitor_SMD:C_0805_2012Metric_Pad1.15x1.40mm_HandSolder" H 5200 2450 50  0001 C CNN
+F 2 "Capacitor_SMD:C_0603_1608Metric_Pad1.05x0.95mm_HandSolder" H 5200 2450 50  0001 C CNN
 F 3 "~" H 5200 2450 50  0001 C CNN
 	1    5200 2450
@@
 F 0 "C7" H 5592 2496 50  0000 L CNN
 F 1 "100n" H 5592 2405 50  0000 L CNN
-F 2 "Capacitor_SMD:C_0805_2012Metric_Pad1.15x1.40mm_HandSolder" H 5500 2450 50  0001 C CNN
+F 2 "Capacitor_SMD:C_0603_1608Metric_Pad1.05x0.95mm_HandSolder" H 5500 2450 50  0001 C CNN
 F 3 "~" H 5500 2450 50  0001 C CNN
 	1    5500 2450
@@
 F 0 "C8" H 5892 2496 50  0000 L CNN
 F 1 "100n" H 5892 2405 50  0000 L CNN
-F 2 "Capacitor_SMD:C_0805_2012Metric_Pad1.15x1.40mm_HandSolder" H 5800 2450 50  0001 C CNN
+F 2 "Capacitor_SMD:C_0603_1608Metric_Pad1.05x0.95mm_HandSolder" H 5800 2450 50  0001 C CNN
 F 3 "~" H 5800 2450 50  0001 C CNN
 	1    5800 2450
@@
 F 0 "C10" H 6192 2496 50  0000 L CNN
 F 1 "100n" H 6192 2405 50  0000 L CNN
-F 2 "Capacitor_SMD:C_0805_2012Metric_Pad1.15x1.40mm_HandSolder" H 6100 2450 50  0001 C CNN
+F 2 "Capacitor_SMD:C_0603_1608Metric_Pad1.05x0.95mm_HandSolder" H 6100 2450 50  0001 C CNN
 F 3 "~" H 6100 2450 50  0001 C CNN
 	1    6100 2450

Commit message: PCB design finished
Parts:
- BT1: footprint TestPoint:TestPoint_2Pads_Pitch2.54mm_Drill0.8mm -> Connector_PinHeader_2.54mm:PinHeader_1x02_P2.54mm_Vertical
Changed lines of the file:
@@
 F 0 "BT1" H 5258 1496 50  0000 L CNN
 F 1 "Battery" H 5258 1405 50  0000 L CNN
-F 2 "TestPoint:TestPoint_2Pads_Pitch2.54mm_Drill0.8mm" V 5150 1510 50  0001 C CNN
+F 2 "Connector_PinHeader_2.54mm:PinHeader_1x02_P2.54mm_Vertical" V 5150 1510 50  0001 C CNN
 F 3 "~" V 5150 1510 50  0001 C CNN
 	1    5150 1450

Commit message: board ready to production
Parts:
- J4: footprint Connector_PinSocket_2.54mm:PinSocket_1x06_P2.54mm_Horizontal -> Connector_PinSocket_2.54mm:PinSocket_1x06_P2.54mm_Vertical
Changed lines of the file:
@@
 F 0 "J4" H 7477 5176 50  0000 L CNN
 F 1 "BLE_Connector" H 7477 5085 50  0000 L CNN
-F 2 "Connector_PinSocket_2.54mm:PinSocket_1x06_P2.54mm_Horizontal" H 7450 5200 50  0001 C CNN
+F 2 "Connector_PinSocket_2.54mm:PinSocket_1x06_P2.54mm_Vertical" H 7450 5200 50  0001 C CNN
 F 3 "~" H 7450 5200 50  0001 C CNN
 	1    7450 5200

Commit message: ready to panelize
Parts:
- added R10: 100K, Resistor_SMD:R_0805_2012Metric_Pad1.15x1.40mm_HandSolder, symbol Device:R_Small
Connections:
- net GND: now also R10.2; no longer U1.60 (BOOT0)
- new net: R10.1, U1.60 (BOOT0)
Changed lines of the file:
@@
 L power:GND #PWR0102
 U 1 1 5B5913D8
-P 1600 1850
-F 0 "#PWR0102" H 1600 1600 50  0001 C CNN
-F 1 "GND" H 1605 1677 50  0000 C CNN
-F 2 "" H 1600 1850 50  0001 C CNN
-F 3 "" H 1600 1850 50  0001 C CNN
-	1    1600 1850
-	1    0    0    -1
-$EndComp
-Wire Wire Line
-	1600 1850 1600 1750
-Wire Wire Line
-	1600 1750 2200 1750
+P 1350 1850
+F 0 "#PWR0102" H 1350 1600 50  0001 C CNN
+F 1 "GND" H 1355 1677 50  0000 C CNN
+F 2 "" H 1350 1850 50  0001 C CNN
+F 3 "" H 1350 1850 50  0001 C CNN
+	1    1350 1850
+	1    0    0    -1
+$EndComp
+Wire Wire Line
+	1350 1850 1350 1750
+Wire Wire Line
+	1350 1750 1500 1750
 $Comp
 L Device:Battery BT1
@@
 Wire Wire Line
 	6650 5100 7250 5100
+$Comp
+L Device:R_Small R10
+U 1 1 5B629FC7
+P 1600 1750
+F 0 "R10" V 1404 1750 50  0000 C CNN
+F 1 "100K" V 1495 1750 50  0000 C CNN
+F 2 "Resistor_SMD:R_0805_2012Metric_Pad1.15x1.40mm_HandSolder" H 1600 1750 50  0001 C CNN
+F 3 "~" H 1600 1750 50  0001 C CNN
+	1    1600 1750
+	0    1    1    0
+$EndComp
+Wire Wire Line
+	1700 1750 2200 1750
 $EndSCHEMATC
